File: eagle/SerialChiller.brd (EAGLE design)
At the start: 56.5 x 30.5 mm, 19 parts, among them IC1 LM1117IMPX-3.3

Commit message: 1.0
Routing:
- net +3V3: track 79.8 -> 78.9 mm
- net GND: vias 57 -> 56
Other:
- outline, holes or cut-outs redrawn
- board text added: "SerialChiller 1.0"
Changed lines of the file:
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@@
 <wire x1="102.5525" y1="41.275" x2="102.5525" y2="12.065" width="0" layer="20"/>
 <wire x1="102.5525" y1="12.065" x2="101.9175" y2="11.43" width="0" layer="20" curve="-90"/>
-<wire x1="101.9175" y1="11.43" x2="87.6935" y2="11.43" width="0" layer="20"/>
+<wire x1="67.6275" y1="13.6525" x2="86.4235" y2="13.6525" width="0" layer="20"/>
+<wire x1="86.4235" y1="13.6525" x2="87.0585" y2="13.0175" width="0" layer="20" curve="-90"/>
+<wire x1="87.0585" y1="13.0175" x2="87.0585" y2="12.065" width="0" layer="20"/>
+<wire x1="87.0585" y1="12.065" x2="87.6935" y2="11.43" width="0" layer="20" curve="90"/>
+<wire x1="87.6935" y1="11.43" x2="101.9175" y2="11.43" width="0" layer="20"/>
 <wire x1="87.6935" y1="41.91" x2="101.9175" y2="41.91" width="0" layer="20"/>
 <wire x1="101.9175" y1="41.91" x2="102.5525" y2="41.275" width="0" layer="20" curve="-90"/>
@@
 <wire x1="84.455" y1="40.64" x2="84.455" y2="40.005" width="0" layer="20"/>
 <wire x1="84.455" y1="40.005" x2="85.09" y2="39.37" width="0" layer="20" curve="90"/>
-<wire x1="83.82" y1="41.275" x2="50.4025" y2="41.275" width="0" layer="20"/>
-<wire x1="50.4025" y1="41.275" x2="46.0375" y2="36.275" width="0" layer="20" curve="90"/>
+<wire x1="83.82" y1="41.275" x2="51.0375" y2="41.275" width="0" layer="20"/>
+<wire x1="51.0375" y1="41.275" x2="46.0375" y2="36.275" width="0" layer="20" curve="90"/>
 <wire x1="46.0375" y1="36.275" x2="46.0375" y2="17.065" width="0" layer="20"/>
 <wire x1="46.0375" y1="17.065" x2="51.0375" y2="12.065" width="0" layer="20" curve="90"/>
 <wire x1="51.0375" y1="12.065" x2="66.3575" y2="12.065" width="0" layer="20"/>
+<wire x1="66.3575" y1="12.065" x2="66.9925" y2="12.7" width="0" layer="20" curve="90"/>
+<wire x1="66.9925" y1="12.7" x2="66.9925" y2="13.0175" width="0" layer="20"/>
+<wire x1="66.9925" y1="13.0175" x2="67.6275" y2="13.6525" width="0" layer="20" curve="-90"/>
 <wire x1="83.82" y1="41.275" x2="84.455" y2="40.64" width="0" layer="20" curve="-90"/>
-<wire x1="66.3575" y1="12.065" x2="66.9925" y2="12.7" width="0" layer="20" curve="90"/>
-<wire x1="66.9925" y1="12.7" x2="66.9925" y2="13.335" width="0" layer="20"/>
-<wire x1="66.9925" y1="13.335" x2="67.6275" y2="13.97" width="0" layer="20" curve="-90"/>
-<wire x1="67.6275" y1="13.97" x2="86.4235" y2="13.97" width="0" layer="20"/>
-<wire x1="86.4235" y1="13.97" x2="87.0585" y2="13.335" width="0" layer="20" curve="-90"/>
-<wire x1="87.0585" y1="13.335" x2="87.0585" y2="12.065" width="0" layer="20"/>
-<wire x1="87.0585" y1="12.065" x2="87.6935" y2="11.43" width="0" layer="20" curve="90"/>
 <hole x="49.53" y="33.9725" drill="3.2"/>
 <hole x="49.53" y="19.3675" drill="3.2"/>
 <circle x="49.53" y="33.9725" radius="2.99999375" width="0.254" layer="48"/>
 <circle x="49.53" y="19.3675" radius="2.99999375" width="0.254" layer="48"/>
+<text x="75.72375" y="36.195" size="1.016" layer="21" font="fixed">SerialChiller 1.0</text>
 </plain>
 <attributes>
@@
 </polygon>
 <via x="53.975" y="27.6225" extent="1-16" drill="0.254"/>
-<via x="80.3275" y="14.9225" extent="1-16" drill="0.254"/>
+<via x="80.16875" y="14.44625" extent="1-16" drill="0.254"/>
 <via x="48.895" y="26.67" extent="1-16" drill="0.254"/>
 <via x="48.895" y="14.605" extent="1-16" drill="0.254"/>
@@
 <via x="89.5223" y="34.58845" extent="1-16" drill="0.254"/>
 <via x="90.4748" y="34.58845" extent="1-16" drill="0.254"/>
-<via x="72.39" y="14.76375" extent="1-16" drill="0.254"/>
+<via x="72.54875" y="14.44625" extent="1-16" drill="0.254"/>
 <contactref element="ESP-WROOM-32" pad="23"/>
-<via x="70.00875" y="16.98625" extent="1-16" drill="0.254"/>
 </signal>
 <signal name="RS232RX">
@@
 <wire x1="57.30875" y1="15.39875" x2="59.055" y2="17.145" width="0.8128" layer="1"/>
 <wire x1="59.055" y1="17.145" x2="68.2625" y2="17.145" width="0.8128" layer="1"/>
-<wire x1="68.2625" y1="17.145" x2="69.37375" y2="18.25625" width="0.8128" layer="1"/>
-<wire x1="69.37375" y1="18.25625" x2="70.64375" y2="18.25625" width="0.8128" layer="1"/>
-<wire x1="70.64375" y1="18.25625" x2="73.50125" y2="15.39875" width="0.8128" layer="1"/>
+<wire x1="68.2625" y1="17.145" x2="71.755" y2="17.145" width="0.8128" layer="1"/>
+<wire x1="71.755" y1="17.145" x2="73.50125" y2="15.39875" width="0.8128" layer="1"/>
 <wire x1="73.50125" y1="15.39875" x2="78.89875" y2="15.39875" width="0.8128" layer="1"/>
 <wire x1="52.705" y1="15.39875" x2="57.30875" y2="15.39875" width="0.8128" layer="1"/>
